File: buck_converter.kicad_pcb (KiCad board)
At the start: 2 copper layers, 43.5 x 23 mm, 24 parts, among them U1 TPS54560DDA

Commit message: "Versión 2"
Parts:
- removed G***: LOGO, Logos:KON_6x6
- added RV1: 250k, Potentiometer_SMD:Potentiometer_Bourns_3214W_Vertical, F.Cu at (181.5, 123.0)
- R5: value 140K -> 33K
Connections:
- R5 pad 2: FB -> Net-(R5-Pad2)
Routing:
- net COMP: track 36.7 -> 45.4 mm
- net Net-(R5-Pad2): track 0.00 -> 6.59 mm, vias 0 -> 2
- net /Vin: track 42.0 -> 35.6 mm
- net FB: track 27.2 -> 33.4 mm, vias 0 -> 2
- net Net-(U1-SW): track 29.1 -> 34.2 mm, vias 2 -> 3
- net /Vout: track 54.0 -> 56.9 mm
- net Net-(U1-BOOT): track 9.51 -> 8.75 mm
- net GND: track 0.35 -> 0.00 mm, vias 33 -> 38
- net Net-(U1-EN): track 21.9 -> 22.2 mm, vias 2 -> 3
Other:
- board text added: "Step DownDC-DC Converter with Eco-mode Vin: 4.5V to 60 V - 5 A"
- board text added: "mh-"
- board text removed: "KON Team"
- board text removed: "Step DownDC-DC Converter withEco-mode Vin: 4.5V to 60 V - 5 A Vout: 12 V"
