File: buck_converter.kicad_sch (KiCad schematic)
At the start: 24 parts, among them U1 TPS54560DDA

Commit message: "Versión 2"
Parts:
- RV1: value 250k -> 200k
Changed lines of the file:
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@@
 			)
 		)
-		(property "Value" "250k"
+		(property "Value" "200k"
 			(at 215.9 99.0599 0)
 			(effects
